File: kicad/nue-pcb.kicad_sch (KiCad schematic)
At the start: 154 parts, among them J1 Conn_01x04, J2 AVR-ISP-6, SW1 ESC, SW10 9, SW101 FN1, SW102 SPACE2.75, SW103 SPACE2.25, SW11 0, SW12 -, SW13 =, SW14 2U BACKSP, SW15 TAB150, SW16 Q, SW17 W, SW18 E, SW19 R, SW2 1, SW20 T, SW21 Y, SW22 U, SW23 I, SW24 O, SW25 P, SW26 CURL_L, SW27 CURL_R, SW28 1U RBKSP, SW29 CAPS, SW3 2, SW30 A, SW31 S, SW32 D, SW33 F, SW34 G, SW35 H, SW36 J, SW37 K, SW38 L, SW39 ;, SW4 3, SW40 ', SW41 PIPE150, SW42 ENTER_ANSI, SW43 LSHIFT225, SW44 ISO_PIPE, SW45 Z, SW46 X, SW47 C, SW48 V, SW49 B, SW5 4, SW50 N, SW51 M, SW52 <, SW53 >, SW54 ?, SW55 RSHIFT275, SW56 FN, SW6 5, SW61 FN2, SW65 1U LBACKSP, SW66 STEPPEDCAPS, SW69 RSHIFT175, SW7 6, SW70 LCTRL150, SW71 LWIN100, SW72 LALT150, SW73 SPACE700, SW74 RALT150, SW75 RWIN100, SW76 RCTRL150, SW8 7, SW9 8, U1 ATmega32U4-MU, Y1 16 MHz

Commit message: replace jst footprint, make 2.75/7/10u holes smaller
Parts:
- SW102: footprint kestralib:MXOnly-2.75U-ReversedStabilizers-NoLED -> kestralib:MX275R
- SW73: footprint kestralib:MXOnly-10U-7U-ReversedStabilizers-NoLED -> kestralib:MX10-7U
Changed lines of the file:
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@@
       (effects (font (size 0.9906 0.9906)))
     )
-    (property "Footprint" "kestralib:MXOnly-10U-7U-ReversedStabilizers-NoLED" (id 2) (at 177.8 137.16 0)
+    (property "Footprint" "kestralib:MX10-7U" (id 2) (at 177.8 137.16 0)
       (effects (font (size 1.27 1.27)) hide)
     )
@@
       (effects (font (size 0.9906 0.9906)))
     )
-    (property "Footprint" "kestralib:MXOnly-2.75U-ReversedStabilizers-NoLED" (id 2) (at 177.8 146.05 0)
+    (property "Footprint" "kestralib:MX275R" (id 2) (at 177.8 146.05 0)
       (effects (font (size 1.27 1.27)) hide)
     )
@@
     )
     (path "/00000000-0000-0000-0000-00005f4ec57c"
-      (reference "SW73") (unit 1) (value "SPACE700") (footprint "kestralib:MXOnly-10U-7U-ReversedStabilizers-NoLED")
+      (reference "SW73") (unit 1) (value "SPACE700") (footprint "kestralib:MX10-7U")
     )
     (path "/00000000-0000-0000-0000-00005f8fdf19"
@@
     )
     (path "/ff493b81-79b2-4f65-a979-cc9ab88a078f"
-      (reference "SW102") (unit 1) (value "SPACE2.75") (footprint "kestralib:MXOnly-2.75U-ReversedStabilizers-NoLED")
+      (reference "SW102") (unit 1) (value "SPACE2.75") (footprint "kestralib:MX275R")
     )
     (path "/1e1c2125-eda8-49f7-9d69-aaf5380dafe1"
